File: hardware/OpenLCD.brd (EAGLE design)
At the start: 45.7 x 30.5 mm, 40 parts, among them Q1 PNP-500mA, Q2 PNP-500mA, Q3 PNP-500mA, U1 ATMEGA328P_TQFP, U2 4BIT-RGB, U3 MIC5205-ADJ, Y2 8MHz

Commit message: Updated SFE logos and flames
To avoid extremely long CAM jobs in eagle 7.2
Parts:
- U$1: device SparkFun:SFE-LOGO-FLAME -> SparkFun-Aesthetics:SFE_LOGO_FLAME_.1
- moved U$1 0.46 mm to (24.1, 14.9)
Changed lines of the file:
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@@
 <?xml version="1.0" encoding="utf-8"?>
 <!DOCTYPE eagle SYSTEM "eagle.dtd">
-<eagle version="7.1.0">
+<eagle version="7.2.0">
 <drawing>
 <settings>
@@
 <attribute name="VALUE" value="0.1uF" x="26.67" y="11.43" size="1.778" layer="27" rot="R225" display="off"/>
 </element>
-<element name="U$1" library="SparkFun" package="SFE-LOGO-FLAME" value="LOGO-SFESK" x="23.749" y="15.113" rot="MR0"/>
+<element name="U$1" library="SparkFun-Aesthetics" package="SFE_LOGO_FLAME_.1" value="LOGO-SFESK" x="24.13" y="14.859" rot="MR0"/>
 <element name="JP6" library="SparkFun-Connectors" package="1X01" value="RESET" x="34.29" y="8.89" rot="R270"/>
 <element name="C1" library="SparkFun-Capacitors" package="0603-CAP" value="0.1uF" x="29.21" y="13.97" rot="R45">

Commit message: Adding Arduino examples. Renaming main firmware.
Parts:
- added C5: 0.1uF, SparkFun-Capacitors:0603-CAP
- added R2: 220, SparkFun-Resistors:0603-RES
- U$1: device SparkFun-Aesthetics:SFE_LOGO_FLAME_.1 -> SparkFun:SFE-LOGO-FLAME
- moved U$4 11.5 mm to (53.3, 24.1)
- moved U$1 0.46 mm to (23.7, 15.1)
Connections:
- new net FILTERED_CONTRAST: C5.2, R2.1, U2.3
- net CONTRAST: now also R2.2; no longer U2.3
- net GND: now also C5.1
Routing:
- net CONTRAST: track 34.5 -> 26.2 mm
Changed lines of the file:
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@@
 <?xml version="1.0" encoding="utf-8"?>
 <!DOCTYPE eagle SYSTEM "eagle.dtd">
-<eagle version="7.2.0">
+<eagle version="7.1.0">
 <drawing>
 <settings>
@@
 <attribute name="VALUE" value="0.1uF" x="26.67" y="11.43" size="1.778" layer="27" rot="R225" display="off"/>
 </element>
-<element name="U$1" library="SparkFun-Aesthetics" package="SFE_LOGO_FLAME_.1" value="LOGO-SFESK" x="24.13" y="14.859" rot="MR0"/>
+<element name="U$1" library="SparkFun" package="SFE-LOGO-FLAME" value="LOGO-SFESK" x="23.749" y="15.113" rot="MR0"/>
 <element name="JP6" library="SparkFun-Connectors" package="1X01" value="RESET" x="34.29" y="8.89" rot="R270"/>
 <element name="C1" library="SparkFun-Capacitors" package="0603-CAP" value="0.1uF" x="29.21" y="13.97" rot="R45">
@@
 <attribute name="VALUE" value="0.1uF" x="29.21" y="13.97" size="1.778" layer="27" rot="R45" display="off"/>
 </element>
-<element name="U$4" library="SparkFun-Aesthetics" package="OSHW-LOGO-S" value="OSHW-LOGOS" x="41.91" y="22.86"/>
+<element name="U$4" library="SparkFun-Aesthetics" package="OSHW-LOGO-S" value="OSHW-LOGOS" x="53.34" y="24.13"/>
 <element name="R5" library="SparkFun-Resistors" package="0603-RES" value="240" x="10.16" y="20.32" rot="R270">
 <attribute name="PROD_ID" value="RES-07849" x="10.16" y="20.32" size="1.778" layer="27" font="vector" ratio="15" rot="R270" display="off"/>
@@
 <element name="TP1" library="SparkFun-Passives" package="PAD.03X.04" value="" x="3.175" y="7.62" rot="MR0"/>
 <element name="TP2" library="SparkFun-Passives" package="PAD.03X.04" value="" x="19.685" y="15.621" rot="MR0"/>
+<element name="R2" library="SparkFun-Resistors" package="0603-RES" value="220" x="39.37" y="22.86">
+<attribute name="PROD_ID" value="RES-00824" x="39.37" y="22.86" size="1.778" layer="27" font="vector" ratio="15" display="off"/>
+</element>
+<element name="C5" library="SparkFun-Capacitors" package="0603-CAP" value="0.1uF" x="39.37" y="24.13" rot="R180">
+<attribute name="PROD_ID" value="CAP-00810" x="39.37" y="24.13" size="1.778" layer="27" font="vector" ratio="15" rot="R180" display="off"/>
+</element>
 </elements>
 <signals>
@@
 <contactref element="JP1" pad="CTS"/>
 <contactref element="Y2" pad="2"/>
+<contactref element="C5" pad="1"/>
 </signal>
 <signal name="RST">
@@
 </signal>
 <signal name="CONTRAST">
-<contactref element="U2" pad="3"/>
 <contactref element="U1" pad="13"/>
 <wire x1="20.107515625" y1="13.191828125" x2="20.8856875" y2="13.97" width="0.254" layer="1"/>
@@
 <wire x1="27.94" y1="13.97" x2="36.83" y2="13.97" width="0.254" layer="16"/>
 <wire x1="36.83" y1="13.97" x2="38.1" y2="15.24" width="0.254" layer="16"/>
-<wire x1="38.1" y1="15.24" x2="38.1" y2="27.94" width="0.254" layer="16"/>
-<wire x1="38.1" y1="27.94" x2="39.37" y2="29.21" width="0.254" layer="16"/>
-<wire x1="39.366" y1="29.343" x2="39.366" y2="29.214" width="0.254" layer="16"/>
-<wire x1="39.366" y1="29.214" x2="39.37" y2="29.21" width="0.254" layer="16"/>
+<contactref element="R2" pad="2"/>
+<wire x1="38.1" y1="15.24" x2="38.1" y2="21.59" width="0.254" layer="16"/>
+<wire x1="38.1" y1="21.59" x2="40.22" y2="22.86" width="0" layer="19" extent="1-16"/>
 </signal>
 <signal name="RS">
@@
 <wire x1="27.94" y1="28.79" x2="26.758" y2="28.79" width="0.254" layer="1"/>
 </signal>
+<signal name="FILTERED_CONTRAST">
+<contactref element="U2" pad="3"/>
+<contactref element="C5" pad="2"/>
+<contactref element="R2" pad="1"/>
+<wire x1="38.52" y1="24.13" x2="39.366" y2="29.343" width="0" layer="19" extent="1-1"/>
+<wire x1="38.52" y1="22.86" x2="38.52" y2="24.13" width="0" layer="19" extent="1-1"/>
+</signal>
 </signals>
